File: Power Bus/Eagle/Power Bus.brd (EAGLE design)
At the start: 240 x 40 mm, 24 parts

Commit message: Add files via upload
Parts:
- removed J17, J18: (no value), my-library:2X8
- added J1, J2: (no value), my-library:2X8
- R1: value 1k -> 560
- R2, R3: value 1k -> 2.2k
- moved J10 175.0 mm to (217.2, 27.9)
- moved J9 175.0 mm to (195.3, 27.9)
- renumbered J11 to J3, J12 to J4, J13 to J5, J14 to J6, J15 to J7, J16 to J8
Connections:
- net +12V: now also J1.7, J1.8, J2.7, J2.8; no longer J17.7, J17.8, J18.7, J18.8
- net +5V: now also J1.5, J1.6, J2.5, J2.6; no longer J17.5, J17.6, J18.5, J18.6
- net -12V: now also J1.15, J1.16, J2.15, J2.16; no longer J17.15, J17.16, J18.15, J18.16
- net CV: now also J1.1, J1.2, J2.1, J2.2; no longer J17.1, J17.2, J18.1, J18.2
- net GATE: now also J1.3, J1.4, J2.3, J2.4; no longer J17.3, J17.4, J18.3, J18.4
- net GND: now also J1.10, J1.11, J1.12, J1.13, J1.14, J1.9, J2.10, J2.11, J2.12, J2.13, J2.14, J2.9; no longer J17.10, J17.11, J17.12, J17.13, J17.14, J17.9, J18.10, J18.11, J18.12, J18.13, J18.14, J18.9
Other:
- board text added: "V1.2"
- board text removed: "FLASK"
- board text removed: "SOUND"
- board text removed: "V1.1"
